Commit message: Fix joints value

File: urdf/Z-Arm_10042C1.urdf (robot description, URDF)
Before this commit: robot Z-Arm_10042C0, 6 links, 5 joints
Joints:
- joint joint3: limit lower=-6.284 upper=6.284 effort=30 velocity=1.571 -> lower=-2.967 upper=2.967 effort=30 velocity=1.571
- joint joint4: limit lower=-6.284 upper=6.284 effort=30 velocity=1.571 -> lower=-18.850 upper=18.850 effort=30 velocity=1.571
