Commit message: Fix: Change model mesh path

File: urdf/Z-Arm_10042C0_moveit2.urdf (robot description, URDF)
Before this commit: robot hitbot, 21 links, 20 joints
Links:
- removed link camera_1_accel_frame
- removed link camera_1_accel_optical_frame
- removed link camera_1_bottom_screw_frame
- removed link camera_1_color_frame
- removed link camera_1_color_optical_frame
- removed link camera_1_depth_frame
- removed link camera_1_depth_optical_frame
- removed link camera_1_gyro_frame
- removed link camera_1_gyro_optical_frame
- removed link camera_1_imu_optical_frame
- removed link camera_1_infra1_frame
- removed link camera_1_infra1_optical_frame
- removed link camera_1_infra2_frame
- removed link camera_1_infra2_optical_frame
- removed link camera_1_link
- link base_link: geometry collision mesh filename=file://$(find hitbot_sim)/meshes/Z-Arm_10042C0/base_link.dae; visual mesh filename=file://$(find hitbot_sim)/meshes/Z-Arm_10042C0/base_link.dae
- link link1: geometry collision mesh filename=file://$(find hitbot_sim)/meshes/Z-Arm_10042C0/link1.dae; visual mesh filename=file://$(find hitbot_sim)/meshes/Z-Arm_10042C0/link1.dae
- link link2: geometry collision mesh filename=file://$(find hitbot_sim)/meshes/Z-Arm_10042C0/link2.dae; visual mesh filename=file://$(find hitbot_sim)/meshes/Z-Arm_10042C0/link2.dae
- link link3: geometry collision mesh filename=file://$(find hitbot_sim)/meshes/Z-Arm_10042C0/link3.dae; visual mesh filename=file://$(find hitbot_sim)/meshes/Z-Arm_10042C0/link3.dae
- link link4: geometry collision mesh filename=file://$(find hitbot_sim)/meshes/Z-Arm_10042C0/link4.dae; visual mesh filename=file://$(find hitbot_sim)/meshes/Z-Arm_10042C0/link4.dae
Joints:
- removed joint camera_1_accel_joint
- removed joint camera_1_accel_optical_joint
- removed joint camera_1_color_joint
- removed joint camera_1_color_optical_joint
- removed joint camera_1_depth_joint
- removed joint camera_1_depth_optical_joint
- removed joint camera_1_gyro_joint
- removed joint camera_1_gyro_optical_joint
- removed joint camera_1_imu_optical_joint
- removed joint camera_1_infra1_joint
- removed joint camera_1_infra1_optical_joint
- removed joint camera_1_infra2_joint
- removed joint camera_1_infra2_optical_joint
- removed joint camera_1_joint
- removed joint camera_1_link_joint
