Commit message: Update humble package

File: config/macro.gazebo.xacro (robot description, xacro)
@@ -2,56 +2,71 @@
 <robot xmlns:xacro="http://www.ros.org/wiki/xacro">
 	<xacro:macro name="hitbot_gazebo" params="namespace:=/">
+    <gazebo>
+      <plugin name="gazebo_ros_joint_state_publisher"
+          filename="libgazebo_ros_joint_state_publisher.so">
+          <update_rate>1000</update_rate>
+          <joint_name>joint1</joint_name>
+          <joint_name>joint2</joint_name>
+          <joint_name>joint3</joint_name>
+          <joint_name>joint4</joint_name>
+      </plugin>
+    </gazebo>
     <!-- Base -->
     <gazebo reference="base_link">
-      <kp>1000000.0</kp>
-      <kd>100.0</kd>
-      <mu1>30.0</mu1>
-      <mu2>30.0</mu2>
-      <maxVel>1.0</maxVel>
-      <minDepth>0.001</minDepth>
+      <turnGravityOff>true</turnGravityOff>
+      <kp>0.0</kp>
+      <kd>0.0</kd>
+      <mu1>0.0</mu1>
+      <mu2>0.0</mu2>
+      <maxVel>0.0</maxVel>
+      <minDepth>0.0</minDepth>
     </gazebo>
     <!-- Link1 -->
     <gazebo reference="link1">
-      <kp>1000000.0</kp>
-      <kd>100.0</kd>
-      <mu1>30.0</mu1>
-      <mu2>30.0</mu2>
-      <maxVel>1.0</maxVel>
-      <minDepth>0.001</minDepth>
+      <turnGravityOff>true</turnGravityOff>
+      <kp>0.0</kp>
+      <kd>0.0</kd>
+      <mu1>0.0</mu1>
+      <mu2>0.0</mu2>
+      <maxVel>0.0</maxVel>
+      <minDepth>0.0</minDepth>
     </gazebo>
     <!-- Link2 -->
     <gazebo reference="link2">
-      <kp>1000000.0</kp>
-      <kd>100.0</kd>
-      <mu1>30.0</mu1>
-      <mu2>30.0</mu2>
-      <maxVel>1.0</maxVel>
-      <minDepth>0.001</minDepth>
+      <turnGravityOff>true</turnGravityOff>
+      <kp>0.0</kp>
+      <kd>0.0</kd>
+      <mu1>0.0</mu1>
+      <mu2>0.0</mu2>
+      <maxVel>0.0</maxVel>
+      <minDepth>0.0</minDepth>
     </gazebo>
     <!-- Link3 -->
     <gazebo reference="link3">
-      <kp>1000000.0</kp>
-      <kd>100.0</kd>
-      <mu1>30.0</mu1>
-      <mu2>30.0</mu2>
-      <maxVel>1.0</maxVel>
-      <minDepth>0.001</minDepth>
+      <turnGravityOff>true</turnGravityOff>
+      <kp>0.0</kp>
+      <kd>0.0</kd>
+      <mu1>0.0</mu1>
+      <mu2>0.0</mu2>
+      <maxVel>0.0</maxVel>
+      <minDepth>0.0</minDepth>
     </gazebo>
     <!-- Link4 -->
     <gazebo reference="link4">
-      <kp>1000000.0</kp>
-      <kd>100.0</kd>
-      <mu1>30.0</mu1>
-      <mu2>30.0</mu2>
-      <maxVel>1.0</maxVel>
-      <minDepth>0.001</minDepth>
+      <turnGravityOff>true</turnGravityOff>
+      <kp>0.0</kp>
+      <kd>0.0</kd>
+      <mu1>0.0</mu1>
+      <mu2>0.0</mu2>
+      <maxVel>0.0</maxVel>
+      <minDepth>0.0</minDepth>
     </gazebo>
-      <!-- ros_control plugin -->
-    <gazebo>
+    <!-- ros_control plugin -->
+    <!-- <gazebo>
       <plugin filename="libgazebo_ros2_control.so" name="gazebo_ros2_control">
+        <parameters>$(find hitbot_sim)/config/hitbot_control.yaml</parameters>
         <robot_sim_type>gazebo_ros2_control/DefaultRobotHWSim</robot_sim_type>
-        <parameters>$(find hitbot_sim)/config/hitbot_control.yaml</parameters>
       </plugin>
-    </gazebo>
+    </gazebo> -->
 	</xacro:macro>
 </robot>

File: config/macro.gazebo_control.xacro (robot description, xacro)
@@ -6,10 +6,10 @@
 		<ros2_control name="GazeboSystem" type="system">
 			<hardware>
-				<plugin>gazebo_ros2_control/DefaultRobotHWSim</plugin>
+				<plugin>gazebo_ros2_control/GazeboSystem</plugin>
 	    	</hardware>
 	    	<joint name="joint1">
 	    		<command_interface name="position">
-	    			<param name="min">-6.2832</param>
-	    			<param name="max">6.2832</param>
+	    			<param name="min">-0.95</param>
+	    			<param name="max">0.0</param>
 	    		</command_interface>
 	    		<state_interface name="position"/>
@@ -19,6 +19,6 @@
 	    	<joint name="joint2">
 	    		<command_interface name="position">
-	    			<param name="min">-6.2832</param>
-	    			<param name="max">6.2832</param>
+	    			<param name="min">-1.571</param>
+	    			<param name="max">1.571</param>
 	    		</command_interface>
 	    		<state_interface name="position"/>
@@ -28,6 +28,6 @@
 	    	<joint name="joint3">
 	    		<command_interface name="position">
-	    			<param name="min">-2.7925</param>
-	    			<param name="max">2.7925</param>
+	    			<param name="min">-6.284</param>
+	    			<param name="max">6.284</param>
 	    		</command_interface>
 	    		<state_interface name="position"/>
@@ -37,6 +37,6 @@
 	    	<joint name="joint4">
 	    		<command_interface name="position">
-	    			<param name="min">-6.2832</param>
-	    			<param name="max">6.2832</param>
+	    			<param name="min">-6.284</param>
+	    			<param name="max">6.284</param>
 	    		</command_interface>
 	    		<state_interface name="position"/>
@@ -44,8 +44,9 @@
 	    		<state_interface name="effort"/>
 	    	</joint>
+		</ros2_control>
 		<gazebo>
 			<plugin name="gazebo_ros2_control" filename="libgazebo_ros2_control.so">
+				<parameters>$(find hitbot_sim)/config/hitbot_control.yaml</parameters>
 				<robot_sim_type>gazebo_ros2_control/DefaultRobotHWSim</robot_sim_type>
-				<parameters>$(find hitbot_sim)/config/hitbot_control.yaml</parameters>
 		    </plugin>
 		</gazebo>

File: urdf/Z-Arm_10042C0.urdf.xacro (robot description, xacro)
@@ -4,156 +4,10 @@
   <xacro:include filename="$(find hitbot_sim)/config/macro.gazebo.xacro" />
 	<xacro:include filename="$(find hitbot_sim)/config/macro.transmission.xacro" />
-  <!-- <xacro:include filename="$(find hitbot_sim)/config/macro.gazebo_control.xacro" /> -->
-    <link name="world"/>
-    <link name="base_link">
-      <inertial>
-        <origin rpy="0 0 0" xyz="-0.0152493195612961 -0.000340773146600589 0.627217436393109"/>
-        <mass value="12.1147491899625"/>
-        <inertia ixx="1.57331650738548" ixy="0.00013876928001303" ixz="-0.00142621285833315" iyy="1.56540260130721" iyz="-0.00396786578401927" izz="0.0545129495020593"/>
-      </inertial>
-      <visual>
-        <origin rpy="0 0 0" xyz="0 0 0"/>
-        <geometry>
-          <mesh filename="file://$(find hitbot_sim)/meshes/Z-Arm_10042C0/base_link.dae"/>
-        </geometry>
-        <material name="">
-          <color rgba="1 1 1 1"/>
-        </material>
-      </visual>
-      <collision>
-        <origin rpy="0 0 0" xyz="0 0 0"/>
-        <geometry>
-          <mesh filename="file://$(find hitbot_sim)/meshes/Z-Arm_10042C0/base_link.dae"/>
-        </geometry>
-      </collision>
-    </link>
-    <joint name="base_joint" type="fixed">
-      <parent link="world"/>
-      <child link="base_link"/>
-      <origin rpy="-1.5708 0 0" xyz="0 0 0"/>
-    </joint>
-    <link name="link1">
-      <inertial>
-        <origin rpy="0 0 0" xyz="0.0814844684502057 -0.000148613714255294 0.0317838791707967"/>
-        <mass value="0.993699801386025"/>
-        <inertia ixx="0.000950142292489542" ixy="-1.44578489991647E-05" ixz="7.33036655063474E-05" iyy="0.0034290254131011" iyz="-2.09106228762866E-06" izz="0.00392515031508005"/>
-      </inertial>
-      <visual>
-        <origin rpy="0 0 0" xyz="0 0 0"/>
-        <geometry>
-          <mesh filename="file://$(find hitbot_sim)/meshes/Z-Arm_10042C0/link1.dae"/>
-        </geometry>
-        <material name="">
-          <color rgba="0.792156862745098 0.819607843137255 0.933333333333333 1"/>
-        </material>
-      </visual>
-      <collision>
-        <origin rpy="0 0 0" xyz="0 0 0"/>
-        <geometry>
-          <mesh filename="file://$(find hitbot_sim)/meshes/Z-Arm_10042C0/link1.dae"/>
-        </geometry>
-      </collision>
-    </link>
-    <joint name="joint1" type="prismatic">
-      <origin rpy="1.5708 0 0" xyz="0 -1.2 0"/>
-      <parent link="base_link"/>
-      <child link="link1"/>
-      <axis xyz="0 0 1"/>
-      <limit effort="300" lower="-0.95" upper="0" velocity="7"/>
-      <dynamics friction="10" />
-    </joint>
-    <link name="link2">
-      <inertial>
-        <origin rpy="0 0 0" xyz="0.111045959309931 2.43604684770394E-05 -0.0314379854113542"/>
-        <mass value="5.85844227294122"/>
-        <inertia ixx="0.00708782289991147" ixy="7.1034720884927E-06" ixz="0.000255328408086295" iyy="0.0470616581346809" iyz="3.5236472788361E-07" izz="0.0503399714879645"/>
-      </inertial>
-      <visual>
-        <origin rpy="0 0 0" xyz="0 0 0"/>
-        <geometry>
-          <mesh filename="file://$(find hitbot_sim)/meshes/Z-Arm_10042C0/link2.dae"/>
-        </geometry>
-        <material name="">
-          <color rgba="1 1 1 1"/>
-        </material>
-      </visual>
-      <collision>
-        <origin rpy="0 0 0" xyz="0 0 0"/>
-        <geometry>
-          <mesh filename="file://$(find hitbot_sim)/meshes/Z-Arm_10042C0/link2.dae"/>
-        </geometry>
-      </collision>
-    </link>
-    <joint name="joint2" type="revolute">
-      <origin rpy="0 0 0" xyz="0.133 0 0"/>
-      <parent link="link1"/>
-      <child link="link2"/>
-      <axis xyz="0 0 1"/>
-      <limit effort="50" lower="-1.571" upper="1.571" velocity="1.571"/>
-      <dynamics friction="0" />
-    </joint>
-    <link name="link3">
-      <inertial>
-        <origin rpy="0 0 0" xyz="0.0953068068304957 1.45953948384313E-13 -0.0226655447402296"/>
-        <mass value="3.43252725336984"/>
-        <inertia ixx="0.00328366639192851" ixy="-1.56304791044749E-14" ixz="5.94905284720721E-05" iyy="0.0233302625835159" iyz="1.47845983740584E-16" izz="0.0254348240065591"/>
-      </inertial>
-      <visual>
-        <origin rpy="0 0 0" xyz="0 0 0"/>
-        <geometry>
-          <mesh filename="file://$(find hitbot_sim)/meshes/Z-Arm_10042C0/link3.dae"/>
-        </geometry>
-        <material name="">
-          <color rgba="1 1 1 1"/>
-        </material>
-      </visual>
-      <collision>
-        <origin rpy="0 0 0" xyz="0 0 0"/>
-        <geometry>
-          <mesh filename="file://$(find hitbot_sim)/meshes/Z-Arm_10042C0/link3.dae"/>
-        </geometry>
-      </collision>
-    </link>
-    <joint name="joint3" type="revolute">
-      <origin rpy="0 0 0" xyz="0.22 0 -0.06799"/>
-      <parent link="link2"/>
-      <child link="link3"/>
-      <axis xyz="0 0 1"/>
-			<limit effort="50" lower="-6.2832" upper="6.2832" velocity="6.2832"/>
-			<dynamics friction="0" />
-    </joint>
-    <link name="link4">
-      <inertial>
-        <origin rpy="0 0 0" xyz="-0.000247759291386207 -7.08258575587396E-12 -0.0209527102025886"/>
-        <mass value="0.120587662892703"/>
-        <inertia ixx="5.0401439482025E-05" ixy="1.41751614431463E-14" ixz="-1.42422376690236E-07" iyy="5.01231671450723E-05" iyz="8.96921067460828E-15" izz="8.90018861873181E-05"/>
-      </inertial>
-      <visual>
-        <origin rpy="0 0 0" xyz="0 0 0"/>
-        <geometry>
-          <mesh filename="file://$(find hitbot_sim)/meshes/Z-Arm_10042C0/link4.dae"/>
-        </geometry>
-        <material name="">
-          <color rgba="1 1 1 1"/>
-        </material>
-      </visual>
-      <collision>
-        <origin rpy="0 0 0" xyz="0 0 0"/>
-        <geometry>
-          <mesh filename="file://$(find hitbot_sim)/meshes/Z-Arm_10042C0/link4.dae"/>
-        </geometry>
-      </collision>
-    </link>
-    <joint name="joint4" type="revolute">
-      <origin rpy="0 0 3.1416" xyz="0.2 0 -0.0284"/>
-      <parent link="link3"/>
-      <child link="link4"/>
-      <axis xyz="0 0 1"/>
-			<limit effort="50" lower="-6.2832" upper="6.2832" velocity="6.2832"/>
-			<dynamics friction="0" />
-    </joint>
+  <xacro:include filename="$(find hitbot_sim)/config/macro.gazebo_control.xacro" />
+      <!-- Import Z-Arm_10042C0 urdf file -->
+  <xacro:include filename="$(find hitbot_sim)/urdf/Z-Arm_10042C1.urdf" />
 		<xacro:hitbot_transmission />
-		<xacro:hitbot_gazebo namespace="" />
-    <!-- <xacro:hitbot_gazebo_control /> -->
+		<xacro:hitbot_gazebo />
+    <xacro:hitbot_gazebo_control />
   </xacro:macro>
 </robot>

File: urdf/Z-Arm_10042C1.urdf (robot description, URDF)
Before this commit: robot Z-Arm_10042C0, 6 links, 5 joints
Links:
- link base_link: geometry collision mesh filename=file://$(find hitbot_sim)/meshes/Z-Arm_10042C0/base_link.dae; visual mesh filename=file://$(find hitbot_sim)/meshes/Z-Arm_10042C0/base_link.dae
- link link1: geometry collision mesh filename=file://$(find hitbot_sim)/meshes/Z-Arm_10042C0/link1.dae; visual mesh filename=file://$(find hitbot_sim)/meshes/Z-Arm_10042C0/link1.dae
- link link2: mass 5.85844227294122 -> 0.085844227294122; geometry collision mesh filename=file://$(find hitbot_sim)/meshes/Z-Arm_10042C0/link2.dae; visual mesh filename=file://$(find hitbot_sim)/meshes/Z-Arm_10042C0/link2.dae
- link link3: mass 3.43252725336984 -> 0.0343252725336984; geometry collision mesh filename=file://$(find hitbot_sim)/meshes/Z-Arm_10042C0/link3.dae; visual mesh filename=file://$(find hitbot_sim)/meshes/Z-Arm_10042C0/link3.dae
- link link4: mass 0.120587662892703 -> 0.0120587662892703; geometry collision mesh filename=file://$(find hitbot_sim)/meshes/Z-Arm_10042C0/link4.dae; visual mesh filename=file://$(find hitbot_sim)/meshes/Z-Arm_10042C0/link4.dae

Commit message: try to upgrade gazebo-classic ->  gazebo-harmonic

File: config/macro.gazebo.xacro (robot description, xacro)
@@ -3,12 +3,7 @@
 	<xacro:macro name="hitbot_gazebo" params="namespace:=/">
     <gazebo>
-      <plugin name="gazebo_ros_joint_state_publisher"
-          filename="libgazebo_ros_joint_state_publisher.so">
-          <update_rate>1000</update_rate>
-          <joint_name>joint1</joint_name>
-          <joint_name>joint2</joint_name>
-          <joint_name>joint3</joint_name>
-          <joint_name>joint4</joint_name>
-      </plugin>
+      <plugin filename="ign_ros2_control-system" name="ign_ros2_control::IgnitionROS2ControlPlugin">
+          <parameters>$(find hitbot_sim)/config/hitbot_control_gz.yaml</parameters>
+        </plugin>
     </gazebo>
     <!-- Base -->

File: config/macro.gazebo_control.xacro (robot description, xacro)
@@ -1,8 +1,8 @@
 <?xml version="1.0"?>
 <robot xmlns:xacro="http://www.ros.org/wiki/xacro">
-	<xacro:macro name="hitbot_gazebo_control">
-		<ros2_control name="GazeboSystem" type="system">
+	<xacro:macro name="hitbot_gz_ros2_control">
+		<ros2_control name="GazeboSimSystem" type="system">
 			<hardware>
-				<plugin>gazebo_ros2_control/GazeboSystem</plugin>
+				<plugin>ign_ros2_control/IgnitionSystem</plugin>
 	    	</hardware>
 	    	<joint name="joint1">
@@ -43,10 +43,4 @@
 	    	</joint>
 		</ros2_control>
-		<gazebo>
-			<plugin name="gazebo_ros2_control" filename="libgazebo_ros2_control.so">
-				<parameters>$(find hitbot_sim)/config/hitbot_control.yaml</parameters>
-				<robot_sim_type>gazebo_ros2_control/DefaultRobotHWSim</robot_sim_type>
-		    </plugin>
-		</gazebo>
 	</xacro:macro>
 </robot>

File: urdf/Z-Arm_10042C0_gazebo_properties.urdf.xacro (robot description, xacro)
@@ -6,14 +6,9 @@
   <xacro:include filename="$(find hitbot_sim)/config/macro.gazebo_control.xacro" />
   <xacro:include filename="$(find hitbot_sim)/urdf/Z-Arm_10042C0_gazebo_sensor_properties.urdf.xacro" />
-  <xacro:include filename="$(find hitbot_sim)/urdf/sensors/d435.urdf.xacro" />
   <!-- Import Z-Arm_10042C0 urdf file -->
   <xacro:include filename="$(find hitbot_sim)/urdf/Z-Arm_10042C0_gazebo.urdf" />
-  <!-- IntelRealsense D435 (Plugin) -->
-  <xacro:sensor_d455 parent="link1" name="camera_1" use_nominal_extrinsics="$(arg use_nominal_extrinsics)">
-    <xacro:insert_block name="camera_1_pose" />
-  </xacro:sensor_d455>
 		<xacro:hitbot_gazebo />
 		<xacro:hitbot_transmission />
-    <xacro:hitbot_gazebo_control />
+    <xacro:hitbot_gz_ros2_control />
   </xacro:macro>
 </robot>

File: urdf/Z-Arm_10042C0_moveit2.urdf (robot description, URDF)
Before this commit: robot hitbot, 21 links, 20 joints
Links:
- link base_link: geometry collision mesh filename=file:///home/roboarm/hitbot_ws/install/hitbot_sim/share/hit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; visual mesh filename=file:///home/roboarm/hitbot_ws/install/hitbot_sim/share/hit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
- link link1: geometry collision mesh filename=file:///home/roboarm/hitbot_ws/install/hitbot_sim/share/hit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; visual mesh filename=file:///home/roboarm/hitbot_ws/install/hitbot_sim/share/hit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
- link link2: geometry collision mesh filename=file:///home/roboarm/hitbot_ws/install/hitbot_sim/share/hit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; visual mesh filename=file:///home/roboarm/hitbot_ws/install/hitbot_sim/share/hit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
- link link3: geometry collision mesh filename=file:///home/roboarm/hitbot_ws/install/hitbot_sim/share/hit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; visual mesh filename=file:///home/roboarm/hitbot_ws/install/hitbot_sim/share/hit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
- link link4: geometry collision mesh filename=file:///home/roboarm/hitbot_ws/install/hitbot_sim/share/hit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; visual mesh filename=file:///home/roboarm/hitbot_ws/install/hitbot_sim/share/hit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
